File: Level_Shifters.sch (KiCad schematic (older format))
At the start: 27 parts, among them Q1 BSS138, Q2 BSS138, Q3 BSS138, Q4 BSS138, Q5 BSS138, Q6 BSS138, Q7 BSS138, Q8 BSS138, Q9 BSS138

Commit message: Makes it SMD based, with smaller connectors
Parts:
- removed Q1, Q2, Q3, Q4, Q5, Q6, Q7, Q8, Q9: BSS138, digikey-footprints:SOT-23-3, symbol dk_Transistors-FETs-MOSFETs-Single:BSS138
- removed R1, R10, R11, R12, R13, R14, R15, R16, R17, R2, R20, R3, R4, R5, R6, R7, R8, R9: 10k, Resistor_THT:R_Axial_DIN0204_L3.6mm_D1.6mm_P7.62mm_Horizontal, symbol Device:R_US
- added U3, U4: 4504, Package_SO:TSSOP-16_4.4x5mm_P0.65mm, symbol 4xxx:4504
Connections:
- net labels added: GND, HV_10, HV_11, HV_12, LV_10, LV_11, LV_12
- wire segments 99 -> 10
