File: Level_Shifters.sch (KiCad schematic (older format))
At the start: 2 parts, among them U3 4504, U4 4504

Commit message: Change mosfets and resistors to arrays
Parts:
- removed U3, U4: 4504, Package_SO:TSSOP-16_4.4x5mm_P0.65mm, symbol 4xxx:4504
- added R1, R2, R3: 10k, Kicad_extra_components:R_0805_2012Metric_Pad1.15x1.40mm_HandSolder, symbol Device:R_US
- added U10, U3, U4, U7, U8, U9: NTJD5121N, Package_TO_SOT_SMD:SOT-363_SC-70-6, symbol Local:NTJD5121N
Connections:
- net labels added: +5V, X_Dir, X_Dir-, X_Enable-, X_Pulse-, X_Step, Y_Dir, Y_Dir-, Y_Enable-, Y_Pulse-, Y_Step, Z_Dir, Z_Dir-, Z_Enable-, Z_Pulse-, Z_Step, ~X_Enable~, ~Y_Enable~, ~Z_Enable~
- net labels removed: HV, HV_1, HV_10, HV_11, HV_12, HV_2, HV_3, HV_4, HV_5, HV_6, HV_7, HV_8, HV_9, LV, LV_1, LV_10, LV_11, LV_12, LV_2, LV_3, LV_4, LV_5, LV_6, LV_7, LV_8, LV_9
- wire segments 10 -> 27
