File: Pwm_Converter.sch (KiCad schematic (older format))
At the start: 9 parts, among them U5 LM358P

Commit message: Renamed Kicad Project, cleanup
Parts:
- C1, C2, C3: footprint Capacitor_THT:C_Rect_L4.6mm_W2.0mm_P2.50mm_MKS02_FKP02 -> Kicad_extra_components:C_Rect_L4.6mm_W2.0mm_P2.50mm_MKS02_FKP02
Changed lines of the file:
@@
 F 0 "C2" H 3142 3596 50  0000 L CNN
 F 1 "10u" H 3142 3505 50  0000 L CNN
-F 2 "Capacitor_THT:C_Rect_L4.6mm_W2.0mm_P2.50mm_MKS02_FKP02" H 3050 3550 50  0001 C CNN
+F 2 "Kicad_extra_components:C_Rect_L4.6mm_W2.0mm_P2.50mm_MKS02_FKP02" H 3050 3550 50  0001 C CNN
 F 3 "~" H 3050 3550 50  0001 C CNN
 F 4 "FG28X5R1E106MRT06" H 3050 3550 50  0001 C CNN "MPN"
@@
 F 0 "C3" H 4692 3046 50  0000 L CNN
 F 1 "10u" H 4692 2955 50  0000 L CNN
-F 2 "Capacitor_THT:C_Rect_L4.6mm_W2.0mm_P2.50mm_MKS02_FKP02" H 4600 3000 50  0001 C CNN
+F 2 "Kicad_extra_components:C_Rect_L4.6mm_W2.0mm_P2.50mm_MKS02_FKP02" H 4600 3000 50  0001 C CNN
 F 3 "~" H 4600 3000 50  0001 C CNN
 F 4 "FG28X5R1E106MRT06" H 4600 3000 50  0001 C CNN "MPN"
@@
 F 0 "C1" H 2792 3246 50  0000 L CNN
 F 1 "10u" H 2792 3155 50  0000 L CNN
-F 2 "Capacitor_THT:C_Rect_L4.6mm_W2.0mm_P2.50mm_MKS02_FKP02" H 2700 3200 50  0001 C CNN
+F 2 "Kicad_extra_components:C_Rect_L4.6mm_W2.0mm_P2.50mm_MKS02_FKP02" H 2700 3200 50  0001 C CNN
 F 3 "~" H 2700 3200 50  0001 C CNN
 F 4 "FG28X5R1E106MRT06" H 2700 3200 50  0001 C CNN "MPN"

Commit message: Makes it SMD based, with smaller connectors
Parts:
- C1, C2, C3: footprint Kicad_extra_components:C_Rect_L4.6mm_W2.0mm_P2.50mm_MKS02_FKP02 -> Capacitor_SMD:C_1206_3216Metric_Pad1.42x1.75mm_HandSolder; Digi-Key_PN 445-181284-1-ND -> 1276-3045-1-ND; MPN FG28X5R1E106MRT06 -> CL31A106MQHNNNE
- R59, R60, R61: footprint Resistor_THT:R_Axial_DIN0204_L3.6mm_D1.6mm_P7.62mm_Horizontal -> Resistor_SMD:R_1206_3216Metric_Pad1.42x1.75mm_HandSolder; Digi-Key_PN S4.7KCACT-ND -> A129818CT-ND; MPN RNMF14FTC4K70 -> CRGCQ1206F4K7
- R62: footprint Resistor_THT:R_Axial_DIN0204_L3.6mm_D1.6mm_P7.62mm_Horizontal -> Resistor_SMD:R_1206_3216Metric_Pad1.42x1.75mm_HandSolder; Digi-Key_PN S10KCACT-ND -> A130183CT-ND; MPN RNMF14FTC10K0 -> CRGCQ1206J10K
- RV1: Digi-Key_PN 1993-1217-ND -> 1993-1217-ND
- U5: footprint digikey-footprints:SOCKET_DIP-8_7.62mm_Conn -> Package_SO:SOIC-8_3.9x4.9mm_P1.27mm; Digi-Key_PN 296-1395-5-ND -> 296-31667-1-ND; MPN LM358P -> LM358ADRG4
- U5: footprint digikey-footprints:SOCKET_DIP-8_7.62mm_Conn -> Package_SO:SOIC-8_3.9x4.9mm_P1.27mm
