File: Pwm_Converter.sch (KiCad schematic (older format))
At the start: 9 parts, among them U5 LM358P

Commit message: Changed wrong GND for limit switches
Parts:
- C1: Spice_Model (none) -> 10u; Spice_Netlist_Enabled (none) -> Y; Spice_Primitive (none) -> C
- R62: Spice_Model (none) -> 10k; Spice_Netlist_Enabled (none) -> Y; Spice_Primitive (none) -> R
- RV1: Spice_Model (none) -> 20k; Spice_Netlist_Enabled (none) -> Y; Spice_Primitive (none) -> R
- U5: Spice_Lib_File (none) -> sim\\LMx58_LM2904.CIR; Spice_Model (none) -> LMX58_LM2904; Spice_Netlist_Enabled (none) -> Y; Spice_Primitive (none) -> X
Changed lines of the file:
@@
 $Descr A4 11693 8268
 encoding utf-8
-Sheet 2 5
+Sheet 4 5
 Title ""
 Date "2020-02-07"
@@
 F 4 "CRGCQ1206J10K" V 5500 1850 50  0001 C CNN "MPN"
 F 5 "A130183CT-ND" V 5500 1850 50  0001 C CNN "Digi-Key_PN"
+F 6 "R" H 5500 1850 50  0001 C CNN "Spice_Primitive"
+F 7 "10k" H 5500 1850 50  0001 C CNN "Spice_Model"
+F 8 "Y" H 5500 1850 50  0001 C CNN "Spice_Netlist_Enabled"
 	1    5500 1850
 	0    1    1    0
@@
 F 4 "CL31A106MQHNNNE" H 2700 3200 50  0001 C CNN "MPN"
 F 5 "1276-3045-1-ND" H 2700 3200 50  0001 C CNN "Digi-Key_PN"
+F 6 "C" H 2700 3200 50  0001 C CNN "Spice_Primitive"
+F 7 "10u" H 2700 3200 50  0001 C CNN "Spice_Model"
+F 8 "Y" H 2700 3200 50  0001 C CNN "Spice_Netlist_Enabled"
 	1    2700 3200
 	-1   0    0    1
@@
 F 4 "1993-1217-ND" H 4850 1850 50  0001 C CNN "Digi-Key_PN"
 F 5 " N6L50T0C-203 " H 4850 1850 50  0001 C CNN "MPN"
+F 6 "R" H 4850 1850 50  0001 C CNN "Spice_Primitive"
+F 7 "20k" H 4850 1850 50  0001 C CNN "Spice_Model"
+F 8 "Y" H 4850 1850 50  0001 C CNN "Spice_Netlist_Enabled"
 	1    4850 1850
 	0    -1   -1   0
@@
 F 11 "Texas Instruments" H 3550 3950 60  0001 L CNN "Manufacturer"
 F 12 "Active" H 3550 4050 60  0001 L CNN "Status"
+F 13 "X" H 3350 2850 50  0001 C CNN "Spice_Primitive"
+F 14 "LMX58_LM2904" H 3350 2850 50  0001 C CNN "Spice_Model"
+F 15 "Y" H 3350 2850 50  0001 C CNN "Spice_Netlist_Enabled"
+F 16 "sim\\LMx58_LM2904.CIR" H 3350 2850 50  0001 C CNN "Spice_Lib_File"
 	1    3350 2850
 	1    0    0    -1
@@
 F 11 "Texas Instruments" H 5600 3850 60  0001 L CNN "Manufacturer"
 F 12 "Active" H 5600 3950 60  0001 L CNN "Status"
+F 13 "X" H 5400 2750 50  0001 C CNN "Spice_Primitive"
+F 14 "LMX58_LM2904" H 5400 2750 50  0001 C CNN "Spice_Model"
+F 15 "Y" H 5400 2750 50  0001 C CNN "Spice_Netlist_Enabled"
+F 16 "sim\\LMx58_LM2904.CIR" H 5400 2750 50  0001 C CNN "Spice_Lib_File"
 	2    5400 2750
 	1    0    0    -1

Commit message: Change mosfets and resistors to arrays
Parts:
- R59, R60, R61, R62: footprint Resistor_SMD:R_1206_3216Metric_Pad1.42x1.75mm_HandSolder -> Kicad_extra_components:R_0805_2012Metric_Pad1.15x1.40mm_HandSolder
Changed lines of the file:
@@
 $Descr A4 11693 8268
 encoding utf-8
-Sheet 4 5
+Sheet 3 6
 Title ""
-Date "2020-02-07"
-Rev "b4"
+Date "2020-02-12"
+Rev "b5"
 Comp "c6p.dev"
 Comment1 ""
@@
 F 0 "R59" V 1745 2950 50  0000 C CNN
 F 1 "4k7" V 1836 2950 50  0000 C CNN
-F 2 "Resistor_SMD:R_1206_3216Metric_Pad1.42x1.75mm_HandSolder" V 1990 2940 50  0001 C CNN
+F 2 "Kicad_extra_components:R_0805_2012Metric_Pad1.15x1.40mm_HandSolder" V 1990 2940 50  0001 C CNN
 F 3 "~" H 1950 2950 50  0001 C CNN
 F 4 "CRGCQ1206F4K7" V 1950 2950 50  0001 C CNN "MPN"
@@
 F 0 "R60" V 2195 2950 50  0000 C CNN
 F 1 "4k7" V 2286 2950 50  0000 C CNN
-F 2 "Resistor_SMD:R_1206_3216Metric_Pad1.42x1.75mm_HandSolder" V 2440 2940 50  0001 C CNN
+F 2 "Kicad_extra_components:R_0805_2012Metric_Pad1.15x1.40mm_HandSolder" V 2440 2940 50  0001 C CNN
 F 3 "~" H 2400 2950 50  0001 C CNN
 F 4 "CRGCQ1206F4K7" V 2400 2950 50  0001 C CNN "MPN"
@@
 F 0 "R61" V 4145 2850 50  0000 C CNN
 F 1 "4k7" V 4236 2850 50  0000 C CNN
-F 2 "Resistor_SMD:R_1206_3216Metric_Pad1.42x1.75mm_HandSolder" V 4390 2840 50  0001 C CNN
+F 2 "Kicad_extra_components:R_0805_2012Metric_Pad1.15x1.40mm_HandSolder" V 4390 2840 50  0001 C CNN
 F 3 "~" H 4350 2850 50  0001 C CNN
 F 4 "CRGCQ1206F4K7" V 4350 2850 50  0001 C CNN "MPN"
@@
 F 0 "R62" V 5295 1850 50  0000 C CNN
 F 1 "10k" V 5386 1850 50  0000 C CNN
-F 2 "Resistor_SMD:R_1206_3216Metric_Pad1.42x1.75mm_HandSolder" V 5540 1840 50  0001 C CNN
+F 2 "Kicad_extra_components:R_0805_2012Metric_Pad1.15x1.40mm_HandSolder" V 5540 1840 50  0001 C CNN
 F 3 "~" H 5500 1850 50  0001 C CNN
 F 4 "CRGCQ1206J10K" V 5500 1850 50  0001 C CNN "MPN"
