File: opto_limits.sch (KiCad schematic (older format))
At the start: 18 parts, among them U1 LTV-847, U2 LTV-847

Commit message: Makes it SMD based, with smaller connectors
Parts:
- R29, R30, R31, R32, R33, R34, R35, R36: footprint Resistor_THT:R_Axial_DIN0204_L3.6mm_D1.6mm_P7.62mm_Horizontal -> Resistor_SMD:R_1206_3216Metric_Pad1.42x1.75mm_HandSolder; Digi-Key_PN S220CACT-ND -> A129802CT-ND; MPN RNMF14FTC220R -> CRGCQ1206F220R
- R37, R38, R39, R40, R41, R42, R43, R44: footprint Resistor_THT:R_Axial_DIN0204_L3.6mm_D1.6mm_P7.62mm_Horizontal -> Resistor_SMD:R_1206_3216Metric_Pad1.42x1.75mm_HandSolder; Digi-Key_PN S4.7KCACT-ND -> A129818CT-ND; MPN RNMF14FTC4K70 -> CRGCQ1206F4K7
- U1, U2: footprint digikey-footprints:Socket_DIP-16_7.62mm_Conn -> Kicad_extra_components:SOIC254P1016X460-16N; Digi-Key_PN 160-1370-5-ND -> 160-1371-5-ND; MPN LTV-847 -> LTV-847S
Connections:
- net labels added: e
- net labels removed: Probe
