File: CNCFia.sch (KiCad schematic (older format))
At the start: 23 parts, among them J1 GND, J10 Driver_X, J11 Driver_Y, J12 Driver_Z, J13 Coolant, J14 Spin_10V, J15 Spin_Enabl, J16 Spin_Dir, J17 Mist, J2 EXT_5V, J3 Limit SW_XY, J4 Limit SW_ZA, J5 Extra SW 0, J6 Extra SW 1, J7 EXT_12V, J8 OPTO_5V, J9 Signal Input, U6 24LC16

Commit message: Fixing schematic symbols
Other:
- note added: "EEPROM"
- moved on the sheet: J3, J4, J5, J6, R5, R6, U6
