File: Relays.sch (KiCad schematic (older format))
At the start: 16 parts, among them Q1 2N3904, Q2 2N3904, Q3 2N3904, Q4 2N3904

Commit message: Change mosfets and resistors to arrays
Parts:
- removed Q1, Q2, Q3, Q4: 2N3904, Package_TO_SOT_SMD:SOT-23_Handsoldering, symbol dk_Transistors-Bipolar-BJT-Single:2N3904
- removed R1, R2, R3, R4: 2k2, Resistor_SMD:R_1206_3216Metric_Pad1.42x1.75mm_HandSolder, symbol Device:R_US
- added U11, U12: NTJD5121N, Package_TO_SOT_SMD:SOT-363_SC-70-6, symbol Local:NTJD5121N
- RLY1, RLY2, RLY3, RLY4: value G5LE-14_DC5 -> G6RL-1 DC5; footprint digikey-footprints:Relay_THT_G5LE-14 -> Kicad_extra_components:RELAY_G6RL-1_5VDC; Digi-Key_PN Z1011-ND -> (none); MPN G5LE-14 DC5 -> G6RL-1 DC5
Connections:
- wire segments 51 -> 48
Other:
- moved on the sheet: D1, D2, D3, D4, RLY1, RLY2, RLY3, RLY4

Commit message: Simplify the power options
Parts:
- RLY1: Digi-Key_PN (none) -> Z2902-ND
- RLY2, RLY3, RLY4: value G6RL-1 DC5 -> G6RL-1 DC5; Digi-Key_PN (none) -> Z2902-ND
Changed lines of the file:
@@
 $Descr A4 11693 8268
 encoding utf-8
-Sheet 2 6
+Sheet 4 6
 Title ""
 Date "2020-02-12"
@@
 F 10 "Omron Electronics Inc-EMC Div" H 5600 2950 60  0001 L CNN "Manufacturer"
 F 11 "Active" H 5600 3050 60  0001 L CNN "Status"
+F 12 "Z2902-ND" H 5400 1850 50  0001 C CNN "Digi-Key_PN"
 	1    5400 1850
 	0    1    1    0
@@
 P 5400 3600
 F 0 "RLY2" V 4935 3600 50  0000 C CNN
-F 1 "G6RL-1 DC5 " V 5026 3600 50  0000 C CNN
+F 1 "G6RL-1 DC5" V 5026 3600 50  0000 C CNN
 F 2 "Kicad_extra_components:RELAY_G6RL-1_5VDC" H 5600 3800 50  0001 L CNN
 F 3 "https://www.mouser.com/datasheet/2/307/en-g6rl-1221008.pdf" H 5600 3900 60  0001 L CNN
@@
 F 10 "Omron Electronics Inc-EMC Div" H 5600 4700 60  0001 L CNN "Manufacturer"
 F 11 "Active" H 5600 4800 60  0001 L CNN "Status"
+F 12 "Z2902-ND" H 5400 3600 50  0001 C CNN "Digi-Key_PN"
 	1    5400 3600
 	0    1    1    0
@@
 P 5400 5400
 F 0 "RLY3" V 4935 5400 50  0000 C CNN
-F 1 "G6RL-1 DC5 " V 5026 5400 50  0000 C CNN
+F 1 "G6RL-1 DC5" V 5026 5400 50  0000 C CNN
 F 2 "Kicad_extra_components:RELAY_G6RL-1_5VDC" H 5600 5600 50  0001 L CNN
 F 3 "https://www.mouser.com/datasheet/2/307/en-g6rl-1221008.pdf" H 5600 5700 60  0001 L CNN
@@
 F 10 "Omron Electronics Inc-EMC Div" H 5600 6500 60  0001 L CNN "Manufacturer"
 F 11 "Active" H 5600 6600 60  0001 L CNN "Status"
+F 12 "Z2902-ND" H 5400 5400 50  0001 C CNN "Digi-Key_PN"
 	1    5400 5400
 	0    1    1    0
@@
 P 5400 7100
 F 0 "RLY4" V 4935 7100 50  0000 C CNN
-F 1 "G6RL-1 DC5 " V 5026 7100 50  0000 C CNN
+F 1 "G6RL-1 DC5" V 5026 7100 50  0000 C CNN
 F 2 "Kicad_extra_components:RELAY_G6RL-1_5VDC" H 5600 7300 50  0001 L CNN
 F 3 "https://www.mouser.com/datasheet/2/307/en-g6rl-1221008.pdf" H 5600 7400 60  0001 L CNN
@@
 F 10 "Omron Electronics Inc-EMC Div" H 5600 8200 60  0001 L CNN "Manufacturer"
 F 11 "Active" H 5600 8300 60  0001 L CNN "Status"
+F 12 "Z2902-ND" H 5400 7100 50  0001 C CNN "Digi-Key_PN"
 	1    5400 7100
 	0    1    1    0
